File: mainboardv1.2.kicad_pcb (KiCad board)
At the start: 2 copper layers, 79.7 x 80 mm, 132 parts, among them IC1 LM2596S, IC2 TDA2822D, IC3 MCP2562P, IC4 STM32F103RBT6, IC5 MIC2288YD5, IC6 ULN2003AD, IC7 LM2901, IC8 REG1117, IC9 SN74LVC1G10, Q1 8MHz

Commit message: Added copyright notice to mask
Parts:
- added svg2mod: G***, Mainboard_v1.2:copyright_mask, B.Cu at (132.2, 77.5)
